Commit message: 使用两轮差速控制机器人-未完成

File: src/glionbot_description/urdf/glionbot/actuator/caster.urdf.xacro (robot description, xacro)
@@ -1,10 +1,17 @@
 <?xml version="1.0"?>
 <robot xmlns:xacro="http://www.ros.org/wiki/xacro">
-    <xacro:macro name="caster_xacro" params="caster_name xyz">
+    <xacro:include filename="$(find  glionbot_description)/urdf/glionbot/common_inertia.xacro" />
+    <xacro:macro name="caster_xacro" params="caster_name xyz r">
+        <gazebo reference="${caster_name}_caster_link">
+            <mu1 value="0.0"/>
+            <mu2 value="0.0"/>
+            <kp value="1000000000.0"/>
+            <kd value="1.0"/>
+        </gazebo>
         <link name="${caster_name}_caster_link">
             <visual>
                 <origin xyz="0.0 0.0 0.0" rpy="0.0 0.0 0.0" />
                 <geometry>
-                    <sphere radius="0.016" />
+                    <sphere radius="${r}" />
                 </geometry>
                 <material name="yellow">
@@ -15,5 +22,5 @@
                 <origin xyz="0.0 0.0 0.0" rpy="0.0 0.0 0.0" />
                 <geometry>
-                    <sphere radius="0.016" />
+                    <sphere radius="${r}" />
                 </geometry>
                 <material name="yellow">
@@ -21,4 +28,5 @@
                 </material>
             </collision>
+            <xacro:sphere_inertia m="0.5" r="${r}" />
         </link>
         <joint name="${caster_name}_caster_joint" type="fixed">

File: src/glionbot_description/urdf/glionbot/actuator/wheel.urdf.xacro (robot description, xacro)
@@ -1,10 +1,11 @@
 <?xml version="1.0"?>
 <robot xmlns:xacro="http://www.ros.org/wiki/xacro">
-    <xacro:macro name="wheel_xacro" params="wheel_name xyz">
+    <xacro:include filename="$(find  glionbot_description)/urdf/glionbot/common_inertia.xacro" />
+    <xacro:macro name="wheel_xacro" params="wheel_name xyz radius length">
         <link name="${wheel_name}_wheel_link">
             <visual>
                 <origin xyz="0.0 0.0 0.0" rpy="1.57079 0.0 0.0" />
                 <geometry>
-                    <cylinder radius="0.032" length="0.04" />
+                    <cylinder radius="${radius}" length="${length}" />
                 </geometry>
                 <material name="yellow">
@@ -15,5 +16,5 @@
                 <origin xyz="0.0 0.0 0.0" rpy="1.57079 0.0 0.0" />
                 <geometry>
-                    <cylinder radius="0.032" length="0.04" />
+                    <cylinder radius="${radius}" length="${length}" />
                 </geometry>
                 <material name="yellow">
@@ -21,4 +22,5 @@
                 </material>
             </collision>
+            <xacro:cylinder_inertia m="0.5" r="${radius}" h="${length}" />
         </link>
         <!-- type="continuous" 该类型关节可以绕某个轴进行无限制旋转-->
@@ -30,4 +32,10 @@
             <axis xyz="0.0 1.0 0.0" />
         </joint>
+        <gazebo reference="${wheel_name}_wheel_link">
+            <mu1 value="20.0"/>
+            <mu2 value="20.0"/>
+            <kp value="100000000000.0"/>
+            <kd value="1.0"/>
+        </gazebo>
     </xacro:macro>
 </robot>

File: src/glionbot_description/urdf/glionbot/base.urdf.xacro (robot description, xacro)
@@ -1,4 +1,5 @@
 <?xml version="1.0"?>
 <robot xmlns:xacro="http://www.ros.org/wiki/xacro">
+    <xacro:include filename="$(find  glionbot_description)/urdf/glionbot/common_inertia.xacro" />
     <xacro:macro name="base_xacro" params="length radius">
         <link name="base_footprint" />
@@ -27,4 +28,5 @@
                 </material>
             </collision>
+            <xacro:cylinder_inertia m="1.0" r="${radius}" h="${length}" />
         </link>
     </xacro:macro>

File: src/glionbot_description/urdf/glionbot/glionbot.urdf.xacro (robot description, xacro)
@@ -11,11 +11,15 @@
     <xacro:base_xacro length="0.12" radius="0.1" />
     <!-- 传感器-->
-    <xacro:imu_xacro xyz="0.0 0.0 0.02" />
+    <xacro:imu_xacro xyz="0.0 0.0 0.02" m="0.5" w="0.02" h="0.02" d="0.02" />
     <xacro:laser_xacro xyz="0.0 0.0 0.10" />
-    <xacro:camera_xacro xyz="0.10 0.0 0.075" />
+    <xacro:camera_xacro xyz="0.10 0.0 0.075" m="0.5" w="0.02" h="0.10" d="0.02" />
     <!-- 执行器主动轮+从动轮-->
-    <xacro:wheel_xacro wheel_name="left" xyz="0.0 0.10 -0.06" />
-    <xacro:wheel_xacro wheel_name="right" xyz="0.0 -0.10 -0.06" />
-    <xacro:caster_xacro caster_name="front" xyz="0.08 0.0 -0.076" />
-    <xacro:caster_xacro caster_name="back" xyz="-0.08 0.0 -0.076" />
+    <xacro:wheel_xacro wheel_name="left" xyz="0.0 0.10 -0.06" radius="0.032" length="0.04" />
+    <xacro:wheel_xacro wheel_name="right" xyz="0.0 -0.10 -0.06" radius="0.032" length="0.04" />
+    <xacro:caster_xacro caster_name="front" xyz="0.08 0.0 -0.076" r="0.016" />
+    <xacro:caster_xacro caster_name="back" xyz="-0.08 0.0 -0.076" r="0.016" />
+    <!-- Gazebo插件-->
+    <xacro:include
+        filename="$(find glionbot_description)/urdf/glionbot/plugins/gazebo_control_plugin.xacro" />
+    <xacro:gazebo_control_plugin />
 </robot>

File: src/glionbot_description/urdf/glionbot/sensor/camera.urdf.xacro (robot description, xacro)
@@ -1,31 +1,33 @@
 <?xml version="1.0"?>
 <robot xmlns:xacro="http://www.ros.org/wiki/xacro">
-    <xacro:macro name="camera_xacro" params="xyz">
+    <xacro:include filename="$(find  glionbot_description)/urdf/glionbot/common_inertia.xacro" />
+    <xacro:macro name="camera_xacro" params="xyz m w h d">
         <!-- 相机模块-->
-         <link name="camera_link">
+        <link name="camera_link">
             <visual>
-                <origin xyz="0.0 0.0 0.0" rpy="0.0 0.0 0.0"/>
+                <origin xyz="0.0 0.0 0.0" rpy="0.0 0.0 0.0" />
                 <geometry>
-                    <box size="0.02 0.10 0.02"/>
+                    <box size="${w} ${h} ${d}" />
                 </geometry>
                 <material name="green">
-                    <color rgba="0.0 1.0 0.0 0.8"/>
+                    <color rgba="0.0 1.0 0.0 0.8" />
                 </material>
             </visual>
             <collision>
-                <origin xyz="0.0 0.0 0.0" rpy="0.0 0.0 0.0"/>
+                <origin xyz="0.0 0.0 0.0" rpy="0.0 0.0 0.0" />
                 <geometry>
-                    <box size="0.02 0.10 0.02"/>
+                    <box size="${w} ${h} ${d}" />
                 </geometry>
                 <material name="green">
-                    <color rgba="0.0 1.0 0.0 0.8"/>
+                    <color rgba="0.0 1.0 0.0 0.8" />
                 </material>
             </collision>
-         </link>
-         <joint name="camera_joint" type="fixed">
-            <parent link="base_link"/>
-            <child link="camera_link"/>
-            <origin xyz="${xyz}"/>
-         </joint>
+            <xacro:box_inertia m="${m}" w="${h}" h="${h}" d="${d}" />
+        </link>
+        <joint name="camera_joint" type="fixed">
+            <parent link="base_link" />
+            <child link="camera_link" />
+            <origin xyz="${xyz}" />
+        </joint>
     </xacro:macro>
 </robot>

File: src/glionbot_description/urdf/glionbot/sensor/imu.urdf.xacro (robot description, xacro)
@@ -1,10 +1,11 @@
 <?xml version="1.0"?>
 <robot xmlns:xacro="http://www.ros.org/wiki/xacro">
-    <xacro:macro name="imu_xacro" params="xyz">
+    <xacro:include filename="$(find  glionbot_description)/urdf/glionbot/common_inertia.xacro" />
+    <xacro:macro name="imu_xacro" params="xyz m w h d">
         <link name="imu_link">
             <visual>
                 <origin xyz="0.0 0.0 0.0" rpy="0.0 0.0 0.0"/>
                 <geometry>
-                    <box size="0.02 0.02 0.02"/>
+                    <box size="${w} ${h} ${d}"/>
                 </geometry>
                 <material name="black">
@@ -15,5 +16,5 @@
                 <origin xyz="0.0 0.0 0.0" rpy="0.0 0.0 0.0"/>
                 <geometry>
-                    <box size="0.02 0.02 0.02"/>
+                    <box size="${w} ${h} ${d}"/>
                 </geometry>
                 <material name="black">
@@ -21,4 +22,5 @@
                 </material>
             </collision>
+            <xacro:box_inertia m="${m}" w="${h}" h="${h}" d="${d}" />
         </link>
         <joint name="imu_joint" type="fixed">

File: src/glionbot_description/urdf/glionbot/sensor/laser.urdf.xacro (robot description, xacro)
@@ -1,5 +1,12 @@
 <?xml version="1.0"?>
 <robot xmlns:xacro="http://www.ros.org/wiki/xacro">
+    <xacro:include filename="$(find  glionbot_description)/urdf/glionbot/common_inertia.xacro" />
     <xacro:macro name="laser_xacro" params="xyz">
+        <gazebo reference="laser_cylinder_link">
+            <material>Gazebo/Black</material>
+        </gazebo>
+        <gazebo reference="laser_link">
+            <material>Gazebo/Black</material>
+        </gazebo>
         <!-- 雷达支撑杆-->
         <link name="laser_cylinder_link">
@@ -22,4 +29,5 @@
                 </material>
             </collision>
+            <xacro:cylinder_inertia m="0.5" r="0.01" h="0.10" />
         </link>
         <joint name="laser_cylinder_joint" type="fixed">
@@ -48,4 +56,5 @@
                 </material>
             </collision>
+            <xacro:cylinder_inertia m="0.5" r="0.02" h="0.02" />
         </link>
         <joint name="laser_joint" type="fixed">
