Commit message: add laser imu camera

File: src/glionbot_description/urdf/glionbot/glionbot.urdf.xacro (robot description, xacro)
@@ -23,3 +23,6 @@
         filename="$(find glionbot_description)/urdf/glionbot/plugins/gazebo_control_plugin.xacro" />
     <xacro:gazebo_control_plugin />
+    <xacro:include
+        filename="$(find glionbot_description)/urdf/glionbot/plugins/gazebo_sensor_plugin.xacro" />
+    <xacro:gazebo_sensor_plugin />
 </robot>

File: src/glionbot_description/urdf/glionbot/sensor/camera.urdf.xacro (robot description, xacro)
@@ -30,4 +30,10 @@
             <origin xyz="${xyz}" />
         </joint>
+        <link name="camera_optical_link"></link>
+        <joint name="camera_optical_joint" type="fixed">
+            <parent link="camera_link"/>
+            <child link="camera_optical_link"/>
+            <origin xyz="0.0 0.0 0.0" rpy="${-pi/2} 0.0 ${-pi/2}"/>
+        </joint>
     </xacro:macro>
 </robot>
